File: pcb/USB-Isolator_v10.brd (EAGLE design)
At the start: 45 x 25 mm, 33 parts, among them IC1 ADUM3160, J1 USB-MICRO, J2 USB-A-AUY1006, U1A RI-0505S, U1B SPU02L-05, X1 PASSER-07, X2 PASSER-07, X3 PASSER-07

Commit message: updated layout and schematics
Parts:
- LOGO3: value LOGO-SPARK_PLACE -> LOGO-S_PLACE_M; device we-symbol:SPARK_TPLACE -> we-symbol:SPARK_TPLACE_M
Connections:
- net D+1 renamed D1_P
- net D+2 renamed D2_P
- net D-1 renamed D1_N
- net D-2 renamed D2_N
Changed lines of the file:
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@@
 </element>
 <element name="LOGO2" library="we-symbol" package="OSHW_6X70" value="OSHW_LOGOX0070" x="31.59125" y="21.9075" smashed="yes"/>
-<element name="LOGO3" library="we-symbol" package="SPARK_TPLACE" value="LOGO-SPARK_PLACE" x="9.8425" y="12.7" smashed="yes"/>
+<element name="LOGO3" library="we-symbol" package="SPARK_TPLACE_M" value="LOGO-S_PLACE_M" x="9.8425" y="12.7" smashed="yes"/>
 <element name="X1" library="we-symbol" package="PASSER_07MM" value="PASSER-07" x="9.525" y="20.955" smashed="yes"/>
 <element name="X2" library="we-symbol" package="PASSER_07MM" value="PASSER-07" x="22.86" y="20.32" smashed="yes"/>
@@
 <contactref element="J2" pad="GND"/>
 <polygon width="0.2032" layer="1" isolate="0.2032">
-<vertex x="26.5" y="25"/>
-<vertex x="26.5" y="0"/>
+<vertex x="26.75" y="25"/>
+<vertex x="26.75" y="0"/>
 <vertex x="45" y="0"/>
 <vertex x="45" y="25"/>
 </polygon>
 <polygon width="0.2032" layer="16" isolate="0.2032">
-<vertex x="26.5" y="25"/>
-<vertex x="26.5" y="0"/>
+<vertex x="26.75" y="25"/>
+<vertex x="26.75" y="0"/>
 <vertex x="45" y="0"/>
 <vertex x="45" y="25"/>
@@
 <via x="37.465" y="24.13" extent="1-16" drill="0.3"/>
 <via x="40.005" y="24.13" extent="1-16" drill="0.3"/>
-<via x="26.9875" y="13.6525" extent="1-16" drill="0.3"/>
-<via x="26.9875" y="11.1125" extent="1-16" drill="0.3"/>
-<via x="26.9875" y="6.0325" extent="1-16" drill="0.3"/>
-<via x="26.9875" y="8.5725" extent="1-16" drill="0.3"/>
-<via x="26.9875" y="3.4925" extent="1-16" drill="0.3"/>
+<via x="27.305" y="13.6525" extent="1-16" drill="0.3"/>
+<via x="27.305" y="11.1125" extent="1-16" drill="0.3"/>
+<via x="27.305" y="6.0325" extent="1-16" drill="0.3"/>
+<via x="27.305" y="8.5725" extent="1-16" drill="0.3"/>
+<via x="27.305" y="3.4925" extent="1-16" drill="0.3"/>
 <via x="32.385" y="0.9525" extent="1-16" drill="0.3"/>
 <via x="34.925" y="0.9525" extent="1-16" drill="0.3"/>
@@
 <contactref element="U1B" pad="5"/>
 <via x="33.3375" y="7.14375" extent="1-16" drill="0.3"/>
-<via x="26.9875" y="18.415" extent="1-16" drill="0.3"/>
+<via x="27.305" y="18.415" extent="1-16" drill="0.3"/>
 <via x="36.195" y="13.335" extent="1-16" drill="0.3"/>
 <contactref element="CU2" pad="1"/>
@@
 <polygon width="0.2032" layer="1" isolate="0.2032">
 <vertex x="0" y="25"/>
-<vertex x="25.5" y="25"/>
-<vertex x="25.5" y="0"/>
+<vertex x="25.25" y="25"/>
+<vertex x="25.25" y="0"/>
 <vertex x="0" y="0"/>
 </polygon>
 <polygon width="0.2032" layer="16" isolate="0.2032">
 <vertex x="0" y="25"/>
-<vertex x="25.5" y="25"/>
-<vertex x="25.5" y="0"/>
+<vertex x="25.25" y="25"/>
+<vertex x="25.25" y="0"/>
 <vertex x="0" y="0"/>
 </polygon>
 <via x="17.145" y="0.9525" extent="1-16" drill="0.3"/>
-<via x="25.0825" y="8.5725" extent="1-16" drill="0.3"/>
-<via x="25.0825" y="6.0325" extent="1-16" drill="0.3"/>
+<via x="24.765" y="8.5725" extent="1-16" drill="0.3"/>
+<via x="24.765" y="6.0325" extent="1-16" drill="0.3"/>
 <via x="19.685" y="0.9525" extent="1-16" drill="0.3"/>
 <via x="9.525" y="24.13" extent="1-16" drill="0.3"/>
@@
 <via x="6.6675" y="11.58875" extent="1-16" drill="0.3"/>
 <via x="0.9525" y="17.78" extent="1-16" drill="0.3"/>
-<via x="25.0825" y="11.1125" extent="1-16" drill="0.3"/>
-<via x="25.0825" y="13.6525" extent="1-16" drill="0.3"/>
+<via x="24.765" y="11.1125" extent="1-16" drill="0.3"/>
+<via x="24.765" y="13.6525" extent="1-16" drill="0.3"/>
 <contactref element="L1" pad="C"/>
 <via x="8.89" y="19.685" extent="1-16" drill="0.3"/>
@@
 <contactref element="U1B" pad="2"/>
 <contactref element="U1A" pad="1"/>
-<via x="25.0825" y="18.415" extent="1-16" drill="0.3"/>
-<via x="25.0825" y="3.4925" extent="1-16" drill="0.3"/>
+<via x="24.765" y="18.415" extent="1-16" drill="0.3"/>
+<via x="24.765" y="3.4925" extent="1-16" drill="0.3"/>
 <via x="13.97" y="15.875" extent="1-16" drill="0.3"/>
 <via x="17.145" y="11.43" extent="1-16" drill="0.3"/>
@@
 <via x="17.145" y="3.01625" extent="1-16" drill="0.3"/>
 </signal>
-<signal name="D-1">
+<signal name="D1_N">
 <contactref element="J1" pad="D-"/>
 <contactref element="R1" pad="1"/>
@@
 <wire x1="11.8325" y1="10.075" x2="11.90625" y2="10.00125" width="0.254" layer="1"/>
 <wire x1="16.66875" y1="5.3975" x2="17.145" y2="5.87375" width="0.254" layer="1"/>
-<wire x1="13.97" y1="5.3975" x2="16.66875" y2="5.3975" width="0.254" layer="1"/>
+<wire x1="16.66875" y1="5.3975" x2="13.97" y2="5.3975" width="0.254" layer="1"/>
 <wire x1="13.97" y1="5.3975" x2="12.22375" y2="6.6675" width="0.254" layer="1" curve="-78.944846"/>
 <wire x1="11.90625" y1="10.00125" x2="11.90625" y2="10.31875" width="0.254" layer="1"/>
@@
 <wire x1="4.785" y1="13.15" x2="8.91625" y2="13.15" width="0.254" layer="1"/>
 </signal>
-<signal name="D+1">
+<signal name="D1_P">
 <contactref element="J1" pad="D+"/>
 <contactref element="R2" pad="1"/>
@@
 <wire x1="4.785" y1="12.5" x2="9.09" y2="12.5" width="0.254" layer="1"/>
 </signal>
-<signal name="D+2">
+<signal name="D2_P">
 <contactref element="R4" pad="2"/>
 <contactref element="J2" pad="D+"/>
@@
 <wire x1="40.3225" y1="13.17625" x2="40.79875" y2="13.17625" width="0.254" layer="1"/>
 </signal>
-<signal name="D-2">
+<signal name="D2_N">
 <contactref element="R3" pad="2"/>
 <contactref element="J2" pad="D-"/>

Commit message: updated schematics
Changed lines of the file:
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@@
 <param name="mvStopFrame" value="1"/>
 <param name="mvCreamFrame" value="0"/>
-<param name="mlMinStopFrame" value="4mil"/>
+<param name="mlMinStopFrame" value="0.3mm"/>
 <param name="mlMaxStopFrame" value="4mil"/>
 <param name="mlMinCreamFrame" value="0mil"/>
