File: pcb/USB-Isolator_v10.sch (EAGLE design)
At the start: 33 parts, among them IC1 ADUM3160, J1 USB-MICRO, J2 USB-A-AUY1006, U1A RI-0505S, U1B SPU02L-05, X1 PASSER-07, X2 PASSER-07, X3 PASSER-07

Commit message: cleaned up schematics and layout
Other:
- note removed: "www.watterott.com"
Changed lines of the file:
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@@
 <setting verticaltext="up"/>
 </settings>
-<grid distance="0.1" unitdist="inch" unit="inch" style="lines" multiple="1" display="no" altdistance="0.01" altunitdist="inch" altunit="inch"/>
+<grid distance="0.05" unitdist="inch" unit="inch" style="lines" multiple="1" display="yes" altdistance="0.025" altunitdist="inch" altunit="inch"/>
 <layers>
 <layer number="1" name="Top" color="4" fill="1" visible="no" active="no"/>
@@
 <sheet>
 <plain>
-<text x="213.36" y="5.08" size="2.54" layer="94" font="vector" align="bottom-right">www.watterott.com</text>
 <text x="158.75" y="8.89" size="2.54" layer="94" rot="R180">Suitable Case: Teko SOAP 1 10006/2</text>
-<text x="161.29" y="31.75" size="1.27" layer="95">Released under the Creative Commons Attribution Share-Alike License</text>
-<text x="161.29" y="29.21" size="1.27" layer="95">http://creativecommons.org/licenses/by-sa/4.0/</text>
-<text x="161.29" y="25.4" size="1.27" layer="95">Designed by Stephan Watterott (Watterott electronic)</text>
+<text x="162.56" y="21.59" size="1.27" layer="95">Released under the Creative Commons Attribution Share-Alike License</text>
+<text x="162.56" y="19.05" size="1.27" layer="95">http://creativecommons.org/licenses/by-sa/4.0/</text>
+<text x="162.56" y="15.24" size="1.27" layer="95">Designed by Stephan Watterott (Watterott electronic)</text>
 <text x="107.95" y="91.44" size="3.81" layer="94">DC/DC Converter</text>
 <text x="114.3" y="151.13" size="3.81" layer="94">USB Isolator</text>
@@
 <instance part="J2" gate="J" x="228.6" y="127"/>
 <instance part="FRAME1" gate="G$1" x="0" y="0"/>
-<instance part="LOGO2" gate="G$1" x="193.04" y="19.05"/>
-<instance part="LOGO3" gate="G$1" x="207.01" y="19.05"/>
-<instance part="X1" gate="X" x="166.37" y="19.05"/>
-<instance part="X2" gate="X" x="173.99" y="19.05"/>
+<instance part="LOGO2" gate="G$1" x="198.12" y="7.62"/>
+<instance part="LOGO3" gate="G$1" x="208.28" y="7.62"/>
+<instance part="X1" gate="X" x="165.1" y="7.62"/>
+<instance part="X2" gate="X" x="170.18" y="7.62"/>
 <instance part="L1" gate="L" x="58.42" y="59.69"/>
 <instance part="R5" gate="R" x="58.42" y="69.85" rot="R90"/>
@@
 <instance part="D2" gate="D" x="190.5" y="119.38"/>
 <instance part="SUPPLY1" gate="G$1" x="190.5" y="106.68"/>
-<instance part="X3" gate="X" x="181.61" y="19.05"/>
+<instance part="X3" gate="X" x="175.26" y="7.62"/>
 </instances>
 <busses>
