File: hardware/USB-Isolator_v10.brd (EAGLE design)
At the start: 45 x 25 mm, 33 parts, among them IC1 ADUM3160, J1 USB-MICRO, J2 USB-A-AUY1006, U1A RI-0505S, U1B SPU02L-05, X1 PASSER-07, X2 PASSER-07, X3 PASSER-07

Commit message: updated layout and schematics
Parts:
- L1: value LED-0603 -> red
Changed lines of the file:
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@@
 <element name="X1" library="we-symbol" package="PASSER_07MM" value="PASSER-07" x="9.525" y="20.955" smashed="yes"/>
 <element name="X2" library="we-symbol" package="PASSER_07MM" value="PASSER-07" x="22.86" y="20.32" smashed="yes"/>
-<element name="L1" library="we-opto" package="LED_0603" value="LED-0603" x="2.8575" y="17.78" smashed="yes" rot="R90">
+<element name="L1" library="we-opto" package="LED_0603" value="red" x="2.8575" y="17.78" smashed="yes" rot="R90">
 <attribute name="NAME" x="5.08" y="17.78" size="0.8128" layer="25" font="vector" ratio="10" align="center"/>
 </element>
